File: PCIE x1 to 2.5G Ethernet.kicad_sch (KiCad schematic)
At the start: 29 parts, among them U1 RTL8125BG-CG, U2 TPS62590DRVT, Y1 25Mhz

Commit message: .
Parts:
- R2: value 280k -> 270k
Changed lines of the file:
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@@
 			)
 		)
-		(property "Value" "280k"
+		(property "Value" "270k"
 			(at 49.53 179.0699 0)
 			(effects
